Commit message: ros2_controll版底盘驱动

File: ros2_ws/src/alohamini_base_control/urdf/alohamini_base.ros2_control.xacro (robot description, xacro)
@@ -17,6 +17,21 @@
   <xacro:arg name="baud_rate" default="1000000"/>
   <xacro:arg name="use_mock_hardware" default="false"/>
+  <!-- Rotation of base_footprint (REP-103: x=forward, y=left) onto the SolidWorks
+       base_link, whose axes are ~90 deg off. Keeps the Odometry arrow aligned with
+       the robot mesh AND with the physical forward direction, so cmd_vel linear.x>0
+       drives the mesh forward (+x) in RViz. -90 verified on this build (base_yaw_deg
+       90 aligned arrow+mesh but pointed them at -x, i.e. driving looked reversed;
+       -90 points them at +x). If it still looks off, try 90 / 180 / 0. -->
+  <xacro:arg name="base_yaw_deg" default="90.0"/>
   <!-- Reuse the existing robot description (meshes, links, joints). -->
   <xacro:include filename="$(find alohamini_description)/urdf/alohamini_nav.urdf"/>
+  <!-- REP-103 root frame. The controller publishes odom -> base_footprint; this
+       static joint rotates it onto base_link so mesh + odometry agree. -->
+  <link name="base_footprint"/>
+  <joint name="base_footprint_joint" type="fixed">
+    <parent link="base_footprint"/>
+    <child link="base_link"/>
+    <origin xyz="0 0 0" rpy="0 0 ${radians($(arg base_yaw_deg))}"/>
+  </joint>
   <ros2_control name="AlohaMiniBase" type="system">
     <hardware>

File: ros2_ws/src/alohamini_description/urdf/alohamini_nav.urdf (robot description, URDF)
Before this commit: robot Aloha, 22 links, 21 joints
Links:
- removed link cad_base_link
- link base_link: mass None -> 5.09802085015176; geometry collision mesh filename=package://alohamini_description/meshes/base_link.STL; visual mesh filename=package://alohamini_description/meshes/base_link.STL
Joints:
- removed joint base_link_to_cad_base_link
- joint base_link_to_imu_frame: origin xyz=0.00978916757496985 0.00084647910851246 0.344753325406094 rpy=0 0 0 -> xyz=0 0 0 rpy=0 0 0
- joint base_link_to_laser_frame: origin xyz=0.20 0 0.12 rpy=0 0 0 -> xyz=0 0 0 rpy=0 0 0
- joint vertical_move: parent cad_base_link -> base_link
- joint wheel1: parent cad_base_link -> base_link
- joint wheel2: parent cad_base_link -> base_link
- joint wheel3: parent cad_base_link -> base_link
