Commit message: docs: 删除无关依赖

File: ros2_ws/src/alohamini_description/urdf/alohamini_nav.urdf (robot description, URDF)
Before this commit: robot Aloha, 21 links, 20 joints
Links:
- added link cad_base_link, mass 5.09802085015176; collision mesh filename=package://alohamini_description/meshes/base_link.STL; visual mesh filename=package://alohamini_description/meshes/base_link.STL
- link base_link: mass 5.09802085015176 -> None; geometry 
Joints:
- added joint base_link_to_cad_base_link: type fixed, parent base_link, child cad_base_link, origin xyz=0 0 0 rpy=0 0 -1.57079632679
- joint base_link_to_imu_frame: origin xyz=0 0 0 rpy=0 0 0 -> xyz=0.00978916757496985 0.00084647910851246 0.344753325406094 rpy=0 0 0
- joint base_link_to_laser_frame: origin xyz=0 0 0 rpy=0 0 0 -> xyz=0.20 0 0.12 rpy=0 0 0
- joint vertical_move: parent base_link -> cad_base_link
- joint wheel1: parent base_link -> cad_base_link
- joint wheel2: parent base_link -> cad_base_link
- joint wheel3: parent base_link -> cad_base_link

Commit message: fix: 修改相关bug

File: ros2_ws/src/alohamini_description/urdf/alohamini_nav.urdf (robot description, URDF)
Before this commit: robot Aloha, 22 links, 21 joints
Joints:
- joint base_link_to_cad_base_link: origin xyz=0 0 0 rpy=0 0 -1.57079632679 -> xyz=0 0 0 rpy=0 0 1.57079632679

Commit message: fix: 座标系修复

File: ros2_ws/src/alohamini_description/urdf/alohamini_nav.urdf (robot description, URDF)
Before this commit: robot Aloha, 21 links, 20 joints
Joints:
- joint base_link_to_laser_frame: origin xyz=0 -0.20 0.12 rpy=0 0 -0.78539816339 -> xyz=0 -0.20 0.12 rpy=0 0 0
